Commit message: new sentry urdf.

File: urdf/sentry/sentry.urdf.xacro (robot description, xacro)
@@ -4,35 +4,38 @@
     <xacro:arg name="load_gimbal" default="true"/>
     <xacro:arg name="load_shooter" default="true"/>
+    <xacro:arg name="camera_link" default="camera_link"/>
+    <xacro:arg name="camera_optical_frame" default="camera_optical_frame"/>
     <xacro:arg name="use_simulation" default="true"/>
+    <xacro:arg name="roller_type" default="realistic"/>
+    <xacro:arg name="oakd_camera_name" default="oak"/>
+    <xacro:arg name="oakd_camera_model" default="OAK-D-PRO"/>
+    <xacro:arg name="base_frame" default="oakd_pro"/>
+    <xacro:arg name="parent_frame" default="yaw"/>
+    <xacro:arg name="cam_pos_x" default="0"/>
+    <xacro:arg name="cam_pos_y" default="0"/>
+    <xacro:arg name="cam_pos_z" default="0.301"/>
+    <xacro:arg name="cam_roll" default="0.0"/>
+    <xacro:arg name="cam_pitch" default="0.41"/>
+    <xacro:arg name="cam_yaw" default="0.0"/>
     <xacro:if value="$(arg load_chassis)">
-        <xacro:include filename="$(find rm_description)/urdf/sentry/chassis.urdf.xacro"/>
-        <xacro:include filename="$(find rm_description)/urdf/sentry/chassis.transmission.urdf.xacro"/>
-        <xacro:chassis use_simulation="$(arg use_simulation)"/>
-    </xacro:if>
-    <xacro:if value="$(arg load_gimbal)">
-        <xacro:include filename="$(find rm_description)/urdf/common/imu.urdf.xacro"/>
-        <xacro:include filename="$(find rm_description)/urdf/common/camera.urdf.xacro"/>
-        <xacro:include filename="$(find rm_description)/urdf/sentry/lower_gimbal.urdf.xacro"/>
-        <xacro:include filename="$(find rm_description)/urdf/sentry/lower_gimbal.transmission.urdf.xacro"/>
-        <xacro:IMU connected_to="lower_pitch" imu_name="lower_gimbal_imu" xyz="0.08 0. 0.08" rpy="${pi} 0 ${pi/2}"/>
-        <xacro:camera_optical_frame xyz="0.085 0.000187 -0.06"
-                                    rpy="-1.6547075 0.0527913 -1.5597212"
-                                    frame_id="lower_camera_optical_frame"
-                                    parent="lower_pitch"
-                                    camera_sim="false"/>
-        <xacro:include filename="$(find rm_description)/urdf/sentry/upper_gimbal.urdf.xacro"/>
-        <xacro:include filename="$(find rm_description)/urdf/sentry/upper_gimbal.transmission.urdf.xacro"/>
-        <xacro:IMU connected_to="upper_pitch" imu_name="upper_gimbal_imu" xyz="0.08 0. 0.08" rpy="0 0 -${pi/2}"/>
-        <xacro:camera_optical_frame xyz="0.1 0.008 0.038"
-                                    rpy="1.8851809 0.0161789 1.5632928"
-                                    frame_id="upper_camera_optical_frame"
-                                    parent="upper_pitch"
-                                    camera_sim="false"/>
-    </xacro:if>
-    <xacro:if value="$(arg load_shooter)">
-        <xacro:include filename="$(find rm_description)/urdf/sentry/upper_shooter.urdf.xacro"/>
-        <xacro:include filename="$(find rm_description)/urdf/sentry/upper_shooter.transmission.urdf.xacro"/>
-        <xacro:include filename="$(find rm_description)/urdf/sentry/lower_shooter.urdf.xacro"/>
-        <xacro:include filename="$(find rm_description)/urdf/sentry/lower_shooter.transmission.urdf.xacro"/>
+        <xacro:include filename="$(find rm_description)/urdf/standard/chassis.urdf.xacro"/>
+        <xacro:chassis roller_type="$(arg roller_type)"/>
+        <xacro:if value="$(arg load_gimbal)">
+            <xacro:include filename="$(find rm_description)/urdf/standard/gimbal.urdf.xacro"/>
+            <xacro:include filename="$(find rm_description)/urdf/sentry/gimbal.transmission.urdf.xacro"/>
+            s
+            <xacro:include filename="$(find rm_description)/urdf/common/imu.urdf.xacro"/>
+            <xacro:include filename="$(find rm_description)/urdf/common/oakd_pro.urdf.xacro"/>
+            <xacro:IMU connected_to="pitch" imu_name="gimbal_imu" xyz="0.08 0. 0.08" rpy="${pi} 0 0"/>
+            <xacro:oak_pro simulation="$(arg use_simulation)" camera_name="$(arg oakd_camera_name)"
+                           parent="$(arg parent_frame)"
+                           camera_model="$(arg oakd_camera_model)" base_frame="$(arg base_frame)"
+                           cam_pos_x="$(arg cam_pos_x)" cam_pos_y="$(arg cam_pos_y)" cam_pos_z="$(arg cam_pos_z)"
+                           cam_roll="$(arg cam_roll)" cam_pitch="$(arg cam_pitch)" cam_yaw="$(arg cam_yaw)"/>
+            <xacro:if value="$(arg load_shooter)">
+                <xacro:include filename="$(find rm_description)/urdf/standard/shooter.urdf.xacro"/>
+                <xacro:include filename="$(find rm_description)/urdf/sentry/shooter.transmission.urdf.xacro"/>
+            </xacro:if>
+        </xacro:if>
     </xacro:if>
     <xacro:if value="$(arg use_simulation)">

File: urdf/sentry/shooter.transmission.urdf.xacro (robot description, xacro)
@@ -1,28 +1,28 @@
 <?xml version="1.0" encoding="utf-8"?>
 <robot>
-    <transmission name="trans_lower_trigger_joint">
+    <transmission name="trans_trigger_joint">
         <type>transmission_interface/SimpleTransmission</type>
-        <actuator name="lower_trigger_joint_motor">
+        <actuator name="trigger_joint_motor">
             <mechanicalReduction>1</mechanicalReduction>
         </actuator>
-        <joint name="lower_trigger_joint">
+        <joint name="trigger_joint">
             <hardwareInterface>hardware_interface/EffortJointInterface</hardwareInterface>
         </joint>
     </transmission>
-    <transmission name="trans_lower_left_friction_wheel_joint_joint">
+    <transmission name="trans_left_friction_wheel_joint">
         <type>transmission_interface/SimpleTransmission</type>
-        <actuator name="lower_left_friction_wheel_joint_motor">
-            <mechanicalReduction>1</mechanicalReduction>
+        <actuator name="left_friction_wheel_joint_motor">
+            <mechanicalReduction>-1</mechanicalReduction>
         </actuator>
-        <joint name="lower_left_friction_wheel_joint">
+        <joint name="left_friction_wheel_joint">
             <hardwareInterface>hardware_interface/EffortJointInterface</hardwareInterface>
         </joint>
     </transmission>
-    <transmission name="trans_lower_right_friction_wheel_joint_joint">
+    <transmission name="trans_right_friction_wheel_joint">
         <type>transmission_interface/SimpleTransmission</type>
-        <actuator name="lower_right_friction_wheel_joint_motor">
-            <mechanicalReduction>1</mechanicalReduction>
+        <actuator name="right_friction_wheel_joint_motor">
+            <mechanicalReduction>-1</mechanicalReduction>
         </actuator>
-        <joint name="lower_right_friction_wheel_joint">
+        <joint name="right_friction_wheel_joint">
             <hardwareInterface>hardware_interface/EffortJointInterface</hardwareInterface>
         </joint>
