Commit message: Delete the supply frame.

File: urdf/sentry/gimbal.urdf.xacro (robot description, xacro)
@@ -33,10 +33,4 @@
         <axis xyz="0 0 1"/>
     </joint>
-    <link name="supply_frame"/>
-    <joint name="supply_joint" type="fixed">
-        <origin xyz="0 0 0" rpy="0 0 ${pi/3}"/>
-        <parent link="yaw"/>
-        <child link="supply_frame"/>
-    </joint>
     <link name="pitch">
         <inertial>
