Commit message: Update some params in the new sentry.

File: urdf/sentry/gimbal.transmission.urdf.xacro (robot description, xacro)
@@ -7,5 +7,5 @@
         </actuator>
         <joint name="yaw_joint">
-            <offset>-0.502</offset>
+            <offset>4.245</offset>
             <hardwareInterface>hardware_interface/EffortJointInterface</hardwareInterface>
         </joint>
@@ -17,14 +17,14 @@
         </actuator>
         <joint name="pitch_joint">
-            <offset>0.523</offset>
+            <offset>0.2427872</offset>
             <hardwareInterface>hardware_interface/EffortJointInterface</hardwareInterface>
         </joint>
     </transmission>
-    <transmission name="trans_cover_joint">
+    <transmission name="trans_barrel_joint">
         <type>transmission_interface/SimpleTransmission</type>
-        <actuator name="cover_joint_motor">
-            <mechanicalReduction>-1</mechanicalReduction>
+        <actuator name="barrel_joint_motor">
+            <mechanicalReduction>1</mechanicalReduction>
         </actuator>
-        <joint name="cover_joint">
+        <joint name="barrel_joint">
             <offset>0</offset>
             <hardwareInterface>hardware_interface/EffortJointInterface</hardwareInterface>

File: urdf/sentry/sentry.urdf.xacro (robot description, xacro)
@@ -6,5 +6,4 @@
     <xacro:arg name="camera_link" default="camera_link"/>
     <xacro:arg name="camera_optical_frame" default="camera_optical_frame"/>
-    <xacro:arg name="roller_type" default="simple"/>
     <xacro:arg name="use_simulation" default="true"/>
     <xacro:arg name="roller_type" default="realistic"/>
@@ -13,12 +12,12 @@
     <xacro:arg name="base_frame" default="oakd_pro"/>
     <xacro:arg name="parent_frame" default="yaw"/>
-    <xacro:arg name="cam_pos_x" default="0"/>
+    <xacro:arg name="cam_pos_x" default="0.059"/>
     <xacro:arg name="cam_pos_y" default="0"/>
-    <xacro:arg name="cam_pos_z" default="0.301"/>
+    <xacro:arg name="cam_pos_z" default="0.352"/>
     <xacro:arg name="cam_roll" default="0.0"/>
-    <xacro:arg name="cam_pitch" default="0.41"/>
+    <xacro:arg name="cam_pitch" default="0.47"/>
     <xacro:arg name="cam_yaw" default="0.0"/>
     <xacro:if value="$(arg load_chassis)">
-        <xacro:include filename="$(find rm_description)/urdf/standard/chassis.urdf.xacro"/>
+        <xacro:include filename="$(find rm_description)/urdf/standard4/chassis.urdf.xacro"/>
         <xacro:chassis roller_type="$(arg roller_type)"/>
         <xacro:if value="$(arg load_gimbal)">
@@ -27,7 +26,6 @@
             <xacro:include filename="$(find rm_description)/urdf/common/camera.urdf.xacro"/>
             <xacro:include filename="$(find rm_description)/urdf/common/imu.urdf.xacro"/>
+            <xacro:include filename="$(find rm_description)/urdf/common/livox_mid360.urdf.xacro"/>
             <xacro:include filename="$(find rm_description)/urdf/common/oakd_pro.urdf.xacro"/>
-            <xacro:camera_sensor xyz="0 0 0.0887" rpy="0 0 0" frame_id="$(arg camera_link)" parent="pitch"
-                                 camera_sim="$(arg use_simulation)"/>
             <xacro:camera_optical_frame xyz="0.06559775176285364 0.000187 0.08746327160978175"
                                         rpy="-1.6347075 0.0527913 -1.5897212"
@@ -38,4 +36,6 @@
                        xyz="0.00246956 0.04105199 -0.07160856"
                        rpy="1.5487827 -0.0054278 -0.01"/>
+            <xacro:livox_mid360 connected_to="yaw" simulation="$(arg use_simulation)" lidar_name="livox_frame"
+                                xyz="0.0 0. 0.286" rpy="${pi} 0 0"/>
             <xacro:oak_pro simulation="$(arg use_simulation)" camera_name="$(arg oakd_camera_name)"
                            parent="$(arg parent_frame)"
@@ -44,5 +44,5 @@
                            cam_roll="$(arg cam_roll)" cam_pitch="$(arg cam_pitch)" cam_yaw="$(arg cam_yaw)"/>
             <xacro:if value="$(arg load_shooter)">
-                <xacro:include filename="$(find rm_description)/urdf/standard/shooter.urdf.xacro"/>
+                <xacro:include filename="$(find rm_description)/urdf/sentry/shooter.urdf.xacro"/>
                 <xacro:include filename="$(find rm_description)/urdf/sentry/shooter.transmission.urdf.xacro"/>
             </xacro:if>

File: urdf/sentry/shooter.transmission.urdf.xacro (robot description, xacro)
@@ -4,8 +4,9 @@
         <type>transmission_interface/SimpleTransmission</type>
         <actuator name="trigger_joint_motor">
-            <mechanicalReduction>1</mechanicalReduction>
+            <mechanicalReduction>-2.5</mechanicalReduction>
         </actuator>
         <joint name="trigger_joint">
             <hardwareInterface>hardware_interface/EffortJointInterface</hardwareInterface>
+            <offset>0.2</offset>
         </joint>
     </transmission>
@@ -13,5 +14,5 @@
         <type>transmission_interface/SimpleTransmission</type>
         <actuator name="left_friction_wheel_joint_motor">
-            <mechanicalReduction>1</mechanicalReduction>
+            <mechanicalReduction>-1</mechanicalReduction>
         </actuator>
         <joint name="left_friction_wheel_joint">
@@ -22,5 +23,5 @@
         <type>transmission_interface/SimpleTransmission</type>
         <actuator name="right_friction_wheel_joint_motor">
-            <mechanicalReduction>1</mechanicalReduction>
+            <mechanicalReduction>-1</mechanicalReduction>
         </actuator>
         <joint name="right_friction_wheel_joint">
